Commit message: Add files via upload

File: urdf/diffbot.urdf (robot description, URDF)
Before this commit: robot diffbot, 3 links, 2 joints
Links:
- link base_link: mass 31.367 -> 7.5332
- link linkleft: mass 1.0462 -> 0.52465
- link linkright: mass 1.0462 -> 0.52465
Joints:
- joint jointleft: origin xyz=-0.13287 0.27 -0.04 rpy=0 0 0 -> xyz=-0.1 0.17 -0.02 rpy=0 0 0
- joint jointright: origin xyz=-0.13287 -0.27 -0.04 rpy=0 0 0 -> xyz=-0.1 -0.17 -0.02 rpy=0 0 0

File: urdf/diffbot_full.xacro (robot description, xacro)
@@ -13,17 +13,22 @@
   <link
     name="base_link">
-    <origin xyz="0.014418 -4.7884E-05 -0.042393" rpy="0 0 0" />
     <inertial>
+      <origin
+        xyz="0.0012511 0 -0.02"
+        rpy="0 0 0" />
       <mass
-        value="31.367" />
+        value="7.5332" />
       <inertia
-        ixx="0.57277"
-        ixy="0.00034867"
-        ixz="0.017425"
-        iyy="1.8106"
-        iyz="-0.00010154"
-        izz="2.3392" />
+        ixx="0.052212"
+        ixy="3.9485E-17"
+        ixz="9.6786E-19"
+        iyy="0.26506"
+        iyz="3.2771E-19"
+        izz="0.31524" />
     </inertial>
     <visual>
+      <origin
+        xyz="0 0 0"
+        rpy="0 0 0" />
       <geometry>
         <mesh
@@ -33,8 +38,11 @@
         name="">
         <color
-          rgba="0.79216 0.81961 0.93333 1" />
+          rgba="0.52941 0.54902 0.54902 1" />
       </material>
     </visual>
     <collision>
+      <origin
+        xyz="0 0 0"
+        rpy="0 0 0" />
       <geometry>
         <mesh
@@ -45,18 +53,22 @@
   <link
     name="linkleft">
-    <origin xyz="-1.3878E-17 -0.01473 3.4694E-18" rpy="0 0 0" />
     <inertial>
-      <origin xyz="-1.3878E-17 -0.01473 3.4694E-18"/>
+      <origin
+        xyz="-1.3878E-17 -0.011048 0"
+        rpy="0 0 0" />
       <mass
-        value="1.0462" />
+        value="0.52465" />
       <inertia
-        ixx="0.0034984"
-        ixy="-1.0646E-19"
-        ixz="-2.2445E-19"
-        iyy="0.006578"
-        iyz="-1.54E-20"
-        izz="0.0034984" />
+        ixx="0.0010699"
+        ixy="2.059E-19"
+        ixz="-1.6414E-19"
+        iyy="0.002062"
+        iyz="9.9564E-21"
+        izz="0.0010699" />
     </inertial>
     <visual>
+      <origin
+        xyz="0 0 0"
+        rpy="0 0 0" />
       <geometry>
         <mesh
@@ -66,8 +78,11 @@
         name="">
         <color
-          rgba="0 0 0 1" />
+          rgba="0.29804 0.29804 0.29804 1" />
       </material>
     </visual>
     <collision>
+      <origin
+        xyz="0 0 0"
+        rpy="0 0 0" />
       <geometry>
         <mesh
@@ -80,5 +95,5 @@
     type="continuous">
     <origin
-      xyz="-0.13287 0.27 -0.04"
+      xyz="-0.1 0.17 -0.02"
       rpy="0 0 0" />
     <parent
@@ -91,17 +106,22 @@
   <link
     name="linkright">
-    <origin xyz="1.3878E-17 0.01473 3.4694E-18" rpy="0 0 0" />
     <inertial>
+      <origin
+        xyz="1.3878E-17 0.011048 0"
+        rpy="0 0 0" />
       <mass
-        value="1.0462" />
+        value="0.52465" />
       <inertia
-        ixx="0.0034984"
-        ixy="-1.0329E-19"
-        ixz="3.236E-35"
-        iyy="0.006578"
-        iyz="-2.1654E-36"
-        izz="0.0034984" />
+        ixx="0.0010699"
+        ixy="1.4008E-19"
+        ixz="1.0434E-35"
+        iyy="0.002062"
+        iyz="5.8775E-36"
+        izz="0.0010699" />
     </inertial>
     <visual>
+      <origin
+        xyz="0 0 0"
+        rpy="0 0 0" />
       <geometry>
         <mesh
@@ -111,8 +131,11 @@
         name="">
         <color
-          rgba="0 0 0 1" />
+          rgba="0.29804 0.29804 0.29804 1" />
       </material>
     </visual>
     <collision>
+      <origin
+        xyz="0 0 0"
+        rpy="0 0 0" />
       <geometry>
         <mesh
@@ -125,5 +148,5 @@
     type="continuous">
     <origin
-      xyz="-0.13287 -0.27 -0.04"
+      xyz="-0.1 -0.17 -0.02"
       rpy="0 0 0" />
     <parent
@@ -134,3 +157,31 @@
       xyz="0 -1 0" />
   </joint>
+  <link name="fcastor_wheel">
+    <origin rpy="0 0 0" xyz="0.00 0 0.00"/>
+    <visual>
+      <geometry>
+        <sphere radius="0.035"/>
+      </geometry>
+      <material
+        name="">
+        <color
+          rgba="0.29804 0.29804 0.29804 1" />
+      </material>
+    </visual>
+    <collision>
+      <geometry>
+        <sphere radius="0.035"/>
+      </geometry>
+    </collision>
+    <inertial>
+      <origin xyz="0 0 0" />
+      <mass value="0.002" />
+      <inertia ixx="0.0001" ixy="0.0" ixz="0.0" iyy="0.0001" iyz="0.0" izz="0.0001" />
+    </inertial>
+  </link>
+  <joint name="base_link__fcastor_wheel" type="continuous">
+    <parent link="base_link"/>
+    <child link="fcastor_wheel"/>
+    <origin xyz="0.2 0 -0.070" rpy="0 0 0"/>
+  </joint>
 </robot>

File: urdf/diffbot_full_gazebo.xacro (robot description, xacro)
@@ -11,5 +11,5 @@
     <kd>10.0</kd>
     <minDepth>0.001</minDepth>
-    <maxVel>0.1</maxVel>
+    <maxVel>1.0</maxVel>
     <fdir1>1 0 0</fdir1>
     <material>Gazebo/FlatBlack</material>
@@ -21,6 +21,15 @@
     <kd>10.0</kd>
     <minDepth>0.001</minDepth>
-    <maxVel>0.1</maxVel>
+    <maxVel>1.0</maxVel>
     <fdir1>1 0 0</fdir1>
+    <material>Gazebo/FlatBlack</material>
+  </gazebo>
+  <gazebo reference="fcastor_wheel">
+    <mu1>0.1</mu1>
+    <mu2>0.1</mu2>
+    <kp>1000000.0</kp>
+    <kd>100.0</kd>
+    <minDepth>0.001</minDepth>
+    <maxVel>1.0</maxVel>
     <material>Gazebo/FlatBlack</material>
   </gazebo>
@@ -31,6 +40,6 @@
       <leftJoint>jointleft</leftJoint>
       <rightJoint>jointright</rightJoint>
-      <wheelSeparation>0.54</wheelSeparation>
-      <wheelDiameter>0.08</wheelDiameter>
+      <wheelSeparation>0.34</wheelSeparation>
+      <wheelDiameter>0.18</wheelDiameter>
       <wheelAcceleration>0.1</wheelAcceleration>
       <wheelTorque>10</wheelTorque>

Commit message: Add files via upload

File: urdf/diffbot.urdf (robot description, URDF)
Before this commit: robot diffbot, 3 links, 2 joints
Links:
- link base_link: mass 7.5332 -> 7.53318560862312
- link linkleft: mass 0.52465 -> 0.524645973149496
- link linkright: mass 0.52465 -> 0.524645973149496
Joints:
- joint jointleft: origin xyz=-0.1 0.17 -0.02 rpy=0 0 0 -> xyz=0 0.17 -0.02 rpy=0 0 0
- joint jointright: origin xyz=-0.1 -0.17 -0.02 rpy=0 0 0 -> xyz=0 -0.17 -0.02 rpy=0 0 0
